Commit message: added velocity controller files

File: omni_description/urdf/velocity_controller.xacro (robot description, xacro)
@@ -1,3 +1,65 @@
 <?xml version="1.0"?>
 <robot name="Omni_bot" xmlns:xacro="http://ros.org/wiki/xacro">
+  <!-- Omnidirectional plugin -->
+  <gazebo>
+    <plugin name="omni_controller_gz" filename="libgazebo_ros_planar_move.so"> <!-- 3 DOF plugin, (Vx,Vy,Wz) -->
+      <command_topic>cmd_vel</command_topic>
+      <odometry_topic>odom</odometry_topic>
+      <odometry_frame>odom</odometry_frame>
+      <robot_base_frame>base_footprint</robot_base_frame>
+      <publish_odom>true</publish_odom>
+      <publish_odom_tf>true</publish_odom_tf>
+      <update_rate>30</update_rate>
+    </plugin>
+  </gazebo>
+  <!-- THIS PLUGIN IS USED TO CORRECTLY VISUALIZED JOINTS POSITION ON RVIZ -->
+  <gazebo>
+    <plugin name="joint_states_gz" filename="libgazebo_ros_joint_state_publisher.so">
+      <ros>
+        <remapping>~/out:=joint_states</remapping>
+      </ros>
+      <update_rate>30</update_rate>
+      <joint_name>front_left_joint</joint_name>
+      <joint_name>front_right_joint</joint_name>
+      <joint_name>back_right_joint</joint_name>
+      <joint_name>back_left_joint</joint_name>
+    </plugin>
+  </gazebo>
+  <!-- PLUGING FOR SERVOMOTORS -->
+  <ros2_control name="GazeboSystem" type="system">
+    <hardware>
+      <plugin>gazebo_ros2_control/GazeboSystem</plugin>
+    </hardware>
+    <!-- List of joints to be controlled -->
+    <joint name="front_left_joint"> <!-- M1 -->
+      <command_interface name="velocity"/>
+      <state_interface name="position"/>
+      <state_interface name="velocity"/>
+      <state_interface name="effort"/>
+    </joint>
+    <joint name="front_right_joint"> <!-- M2 -->
+      <command_interface name="velocity"/>
+      <state_interface name="position"/>
+      <state_interface name="velocity"/>
+      <state_interface name="effort"/>
+    </joint>
+    <joint name="back_right_joint"> <!-- M3 -->
+      <command_interface name="velocity"/>
+      <state_interface name="position"/>
+      <state_interface name="velocity"/>
+      <state_interface name="effort"/>
+    </joint>
+    <joint name="back_left_joint"> <!-- M4 -->
+      <command_interface name="velocity"/>
+      <state_interface name="position"/>
+      <state_interface name="velocity"/>
+      <state_interface name="effort"/>
+    </joint>
+  </ros2_control>
+  <gazebo>
+    <!-- ROS 2 control plugin -->
+    <plugin name="gazebo_ros2_control" filename="libgazebo_ros2_control.so">
+      <parameters>$(find ${package_name})/config/omni_velocity_controller.yaml</parameters>
+    </plugin>
+  </gazebo>
 </robot>
