Commit message: separate urdf sensor link's

File: omni_description/urdf/camera_sensor.xacro (robot description, xacro)
@@ -2,5 +2,32 @@
 <!--Aqui comienza el robot-->
 <robot name="robot_scara" xmlns:xacro="http://ros.org/wiki/xacro" >
-  <gazebo reference="Camera_optical_link">
+  <link name="camera_link">
+      <inertial>
+          <origin xyz="0 0 0" rpy="0 0 0"/>
+          <mass value="0"/>
+          <inertia ixx="0" ixy="0" ixz="0" iyy="0" iyz="0" izz="0"/>
+      </inertial>
+      <visual>
+          <origin xyz="0 0 0" rpy="0 0 0"/>
+          <geometry>
+              <mesh filename="package://omni_description/meshes/sensor/visual/camera_link.STL"/>
+          </geometry>
+          <material name="">
+              <color rgba="0.7 0.7 0.7 1"/>
+          </material>
+      </visual>
+      <collision>
+          <origin xyz="0 0 0" rpy="0 0 0"/>
+          <geometry>
+              <mesh filename="package://omni_description/meshes/sensor/visual/camera_link.STL"/>
+          </geometry>
+      </collision>
+  </link>
+  <joint name="camera_joint" type="fixed">
+      <origin xyz="0.057105 1.7948E-05 0.03755" rpy="0 0 0"/>
+      <parent link="base_link"/>
+      <child link="camera_link"/>
+  </joint>
+  <gazebo reference="camera_link">
     <sensor type="depth" name="camera">
       <always_on>true</always_on>
@@ -34,5 +61,5 @@
             </ros>
             <camera_name>camera</camera_name>
-            <frame_name>P</frame_name>
+            <frame_name>camera_link</frame_name>
             <hack_baseline>0.2</hack_baseline>
         </plugin>

File: omni_description/urdf/lidar_sensor.xacro (robot description, xacro)
@@ -2,4 +2,32 @@
 <robot name="omni_bot" xmlns:xacro="http://ros.org/wiki/xacro">
   <xacro:arg name="laser_visual"  default="true"/> <!-- With true, blue rays are shown in Gazebo-->
+      <link name="laser_link">
+        <inertial>
+            <origin xyz="-0.0176558922685589 0.000671805271544437 0.0219302095894866" rpy="0 0 0" />
+            <mass value="0.0483909504209895" />
+            <inertia ixx="1.58456966399128E-05" ixy="-4.23913983850005E-07" ixz="-2.09597897904374E-07"
+                     iyy="3.89262522903605E-05" iyz="3.24809725932687E-07" izz="4.86230801106223E-05" />
+        </inertial>
+        <visual>
+            <origin xyz="0 0 0" rpy="0 0 0"/>
+            <geometry>
+                <mesh filename="package://omni_description/meshes/sensor/visual/laser_link.STL"/>
+            </geometry>
+            <material name="">
+                <color rgba="0.7 0.7 0.7 1"/>
+            </material>
+        </visual>
+        <collision>
+            <origin xyz="0 0 0" rpy="0 0 0"/>
+            <geometry>
+                <mesh filename="package://omni_description/meshes/sensor/visual/laser_link.STL"/>
+            </geometry>
+        </collision>
+    </link>
+    <joint name="laser_joint" type="fixed">
+        <origin xyz="0.0435 5.25826986680105E-05 0.11" rpy="0 0 0"/>
+        <parent link="base_link"/>
+        <child link="laser_link"/>
+    </joint>
   <gazebo reference="laser_link">
     <sensor type="ray" name="lidar">

File: omni_description/urdf/omni_urdf.xacro (robot description, xacro)
@@ -2,5 +2,4 @@
 <robot name="Omni_bot" xmlns:xacro="http://ros.org/wiki/xacro">
     <link name="base_footprint"/>
-    <link name="imu_link"/>
     <link name="base_link">
         <inertial>
@@ -35,9 +34,4 @@
         <child link="base_link"/>
         <origin xyz="0.0 0.0 0.0815" rpy="0 0 0"/>
-    </joint>
-    <joint name="base_imu" type="fixed">
-        <parent link="base_link"/>
-        <child link="imu_link"/>
-        <origin xyz="-0.06 0.01 0.01" rpy="0 3.1415 1.5707"/>
     </joint>
     <link name="front_right_wheel">
@@ -161,58 +155,3 @@
         <limit effort="100" velocity="1"/>
     </joint>
-    <link name="laser_link">
-        <inertial>
-            <origin xyz="-0.0176558922685589 0.000671805271544437 0.0219302095894866" rpy="0 0 0" />
-            <mass value="0.0483909504209895" />
-            <inertia ixx="1.58456966399128E-05" ixy="-4.23913983850005E-07" ixz="-2.09597897904374E-07"
-                     iyy="3.89262522903605E-05" iyz="3.24809725932687E-07" izz="4.86230801106223E-05" />
-        </inertial>
-        <visual>
-            <origin xyz="0 0 0" rpy="0 0 0"/>
-            <geometry>
-                <mesh filename="package://omni_description/meshes/sensor/visual/laser_link.STL"/>
-            </geometry>
-            <material name="">
-                <color rgba="0.7 0.7 0.7 1"/>
-            </material>
-        </visual>
-        <collision>
-            <origin xyz="0 0 0" rpy="0 0 0"/>
-            <geometry>
-                <mesh filename="package://omni_description/meshes/sensor/visual/laser_link.STL"/>
-            </geometry>
-        </collision>
-    </link>
-    <joint name="laser_joint" type="fixed">
-        <origin xyz="0.0435 5.25826986680105E-05 0.11" rpy="0 0 0"/>
-        <parent link="base_link"/>
-        <child link="laser_link"/>
-    </joint>
-    <link name="camera_link">
-        <inertial>
-            <origin xyz="0 0 0" rpy="0 0 0"/>
-            <mass value="0"/>
-            <inertia ixx="0" ixy="0" ixz="0" iyy="0" iyz="0" izz="0"/>
-        </inertial>
-        <visual>
-            <origin xyz="0 0 0" rpy="0 0 0"/>
-            <geometry>
-                <mesh filename="package://omni_description/meshes/sensor/visual/camera_link.STL"/>
-            </geometry>
-            <material name="">
-                <color rgba="0.7 0.7 0.7 1"/>
-            </material>
-        </visual>
-        <collision>
-            <origin xyz="0 0 0" rpy="0 0 0"/>
-            <geometry>
-                <mesh filename="package://omni_description/meshes/sensor/visual/camera_link.STL"/>
-            </geometry>
-        </collision>
-    </link>
-    <joint name="camera_joint" type="fixed">
-        <origin xyz="0.057105 1.7948E-05 0.03755" rpy="0 0 0"/>
-        <parent link="base_link"/>
-        <child link="camera_link"/>
-    </joint>
 </robot>

File: omni_description/urdf/omni_velocity_controller.xacro (robot description, xacro)
@@ -7,3 +7,4 @@
     <xacro:include filename="$(find ${package_name})/urdf/lidar_sensor.xacro"/>
     <xacro:include filename="$(find ${package_name})/urdf/camera_sensor.xacro"/>
+    <xacro:include filename="$(find ${package_name})/urdf/imu_sensor.xacro"/>
 </robot>

Commit message: fixed camera point cloud

File: omni_description/urdf/camera_sensor.xacro (robot description, xacro)
@@ -28,4 +28,11 @@
       <parent link="base_link"/>
       <child link="camera_link"/>
+  </joint>
+  <link name="camera_PC_link">
+  </link>
+  <joint name="camera_PC_joint" type="fixed">
+      <origin xyz="0.0 0.0 0.0" rpy="-1.57 0 -1.57"/>
+      <parent link="camera_link"/>
+      <child link="camera_PC_link"/>
   </joint>
   <gazebo reference="camera_link">
@@ -61,5 +68,5 @@
             </ros>
             <camera_name>camera</camera_name>
-            <frame_name>camera_link</frame_name>
+            <frame_name>camera_PC_link</frame_name>
             <hack_baseline>0.2</hack_baseline>
         </plugin>

Commit message: reordering urdf files and adding xacro_properties.xacro file to omni_description

File: omni_description/urdf/camera_sensor.xacro (robot description, xacro)
@@ -25,5 +25,5 @@
   </link>
   <joint name="camera_joint" type="fixed">
-      <origin xyz="0.057105 1.7948E-05 0.03755" rpy="0 0 0"/>
+      <origin xyz="${camera_joint_xyz}" rpy="${camera_joint_rpy}"/>
       <parent link="base_link"/>
       <child link="camera_link"/>

File: omni_description/urdf/imu_sensor.xacro (robot description, xacro)
@@ -5,5 +5,5 @@
         <parent link="base_link"/>
         <child link="imu_link"/>
-        <origin xyz="-0.06 0.01 0.01" rpy="0 3.1415 1.5707"/>
+        <origin xyz="${imu_joint_xyz}" rpy="${imu_joint_rpy}"/>
     </joint>
     <gazebo reference="imu_link">

File: omni_description/urdf/lidar_sensor.xacro (robot description, xacro)
@@ -26,5 +26,5 @@
     </link>
     <joint name="laser_joint" type="fixed">
-        <origin xyz="0.0435 5.25826986680105E-05 0.11" rpy="0 0 0"/>
+        <origin xyz="${laser_joint_xyz}" rpy="${laser_joint_rpy}"/>
         <parent link="base_link"/>
         <child link="laser_link"/>

File: omni_description/urdf/omni_velocity_controller.xacro (robot description, xacro)
@@ -5,4 +5,5 @@
     <xacro:include filename="$(find ${package_name})/urdf/omni_gz_properties.xacro"/>
     <xacro:include filename="$(find ${package_name})/urdf/velocity_controller.xacro"/>
+    <xacro:include filename="$(find ${package_name})/urdf/xacro_properties.xacro"/>
     <xacro:include filename="$(find ${package_name})/urdf/lidar_sensor.xacro"/>
     <xacro:include filename="$(find ${package_name})/urdf/camera_sensor.xacro"/>
