Commit message: added sensor descriptions

File: omni_description/urdf/lidar_sensor.xacro (robot description, xacro)
@@ -33,7 +33,10 @@
         </ros>
         <output_type>sensor_msgs/LaserScan</output_type>
-        <frame_name>P</frame_name>
+        <frame_name>laser_link</frame_name>
       </plugin>
     </sensor>
   </gazebo>
+      <gazebo reference="laser_link" >
+        <material>Gazebo/Blue</material>
+    </gazebo>
 </robot>

File: omni_description/urdf/omni_velocity_controller.xacro (robot description, xacro)
@@ -3,5 +3,7 @@
     <xacro:property name="package_name" value="omni_description" />
     <xacro:include filename="$(find ${package_name})/urdf/omni_urdf.xacro"/>
+    <xacro:include filename="$(find ${package_name})/urdf/omni_gz_properties.xacro"/>
     <xacro:include filename="$(find ${package_name})/urdf/velocity_controller.xacro"/>
     <xacro:include filename="$(find ${package_name})/urdf/lidar_sensor.xacro"/>
+    <xacro:include filename="$(find ${package_name})/urdf/camera_sensor.xacro"/>
 </robot>

Commit message: Added gazebo material in lidar_sensor.xacro file

File: omni_description/urdf/lidar_sensor.xacro (robot description, xacro)
@@ -66,5 +66,5 @@
   </gazebo>
       <gazebo reference="laser_link" >
-        <material>Gazebo/Blue</material>
+        <material>Gazebo/Grey</material>
     </gazebo>
 </robot>
