Commit message: Added gazebo material for the base_link in omni_gz_properties.xacro file

File: omni_description/urdf/omni_gz_properties.xacro (robot description, xacro)
@@ -1,4 +1,7 @@
 <?xml version="1.0"?>
 <robot name="Omni_bot" xmlns:xacro="http://ros.org/wiki/xacro">
+    <gazebo reference="camera_link">
+        <material>Gazebo/Grey</material>
+    </gazebo>
     <gazebo reference="base_link">
         <mu1>0.1</mu1>
@@ -9,5 +12,5 @@
         <maxVel>0.1</maxVel>
         <fdir1>1 0 0</fdir1>
-        <material>Gazebo/Red</material>
+        <material>Gazebo/Green</material>
     </gazebo>
     <gazebo reference="front_left_wheel">
