Commit message: add pkg omni_dofbot_description, update dofbot_description and omni_dofbot_bringup

File: dofbot_description/urdf/dofbot_arm_urdf.xacro (robot description, xacro)
@@ -1,4 +1,4 @@
 <?xml version="1.0" encoding="UTF-8" ?>
-<robot name="dofbot_arm">
+<robot name="dofbot_arm" xmlns:xacro="http://ros.org/wiki/xacro">
  <!--Material definition-->
     <material name="eerie_black">
@@ -19,5 +19,5 @@
  <!--Dofbot description-->
     <!--Dofbot Arm Base Link-->
-    <link name="base_link">
+    <link name="arm_base_link">
         <visual>
             <origin xyz="0.0 0.0 0.0" rpy="0.0 0.0 0.0" />
@@ -63,5 +63,5 @@
     <joint name="arm_joint_01" type="revolute">
         <origin xyz="0 0 0.06605" rpy="-0.010805 0 1.5" />
-        <parent link="base_link" />
+        <parent link="arm_base_link" />
         <child link="arm_link_01" />
         <axis xyz="0 0 1" />
@@ -367,5 +367,5 @@
  <!--Gazebo definition-->
     <!--Dofbot-->
-    <gazebo reference="base_link">
+    <gazebo reference="arm_base_link">
         <material>Gazebo/Black</material>
     </gazebo>

Commit message: Added dofbot_bringup package, that include an trajectory controller launch and trajectory test, added a monocular camera for dofbot. Updated dofbot_description, added config for dofbot_trajectory_controller and updated xacro files.

File: dofbot_description/urdf/dofbot_arm_urdf.xacro (robot description, xacro)
@@ -365,184 +365,40 @@
         <mimic joint="grip_joint" multiplier="-1" />
     </joint>
- <!--Gazebo definition-->
-    <!--Dofbot-->
-    <gazebo reference="arm_base_link">
-        <material>Gazebo/Black</material>
-    </gazebo>
-    <gazebo reference="arm_link_01">
-        <material>Gazebo/Green</material>
-    </gazebo>
-    <gazebo reference="arm_link_02">
-        <material>Gazebo/Green</material>
-    </gazebo>
-    <gazebo reference="arm_link_03">
-        <material>Gazebo/Green</material>
-    </gazebo>
-    <gazebo reference="arm_link_04">
-        <material>Gazebo/Green</material>
-    </gazebo>
-    <gazebo reference="arm_link_05">
-        <material>Gazebo/Green</material>
-    </gazebo>
-    <!--Gripper-->
-    <gazebo reference="rgrip_finger01">
-        <material>Gazebo/Grey</material>
-    </gazebo>
-    <gazebo reference="rgrip_finger02">
-        <material>Gazebo/Grey</material>
-    </gazebo>
-    <gazebo reference="rgrip_finger03">
-        <material>Gazebo/Grey</material>
-    </gazebo>
-    <gazebo reference="lgrip_finger01">
-        <material>Gazebo/Grey</material>
-    </gazebo>
-    <gazebo reference="lgrip_finger02">
-        <material>Gazebo/Grey</material>
-    </gazebo>
-    <gazebo reference="lgrip_finger03">
-        <material>Gazebo/Grey</material>
-    </gazebo>
- <!--Sensing-->
     <!-- Mono - camera sensor -->
     <link name="mono_link">
         <inertial>
-            <origin xyz="5.8458E-05 0.0095015 -0.0014824" rpy="0 0 0" />
-            <mass value="0.0097589" />
-            <inertia ixx="3.3488E-06" ixy="1.3667E-08" ixz="6.4235E-09" iyy="1.8662E-06" iyz="-1.0265E-07" izz="2.5696E-06" />
-        </inertial>
-        <visual>
-            <origin xyz="0 0 0" rpy="0 0 0" />
-            <geometry>
-                <mesh filename="package://dofbot_description/meshes/sensor/visual/mono_link.STL" />
-            </geometry>
-            <material name="oxford_blue" />
-        </visual>
-        <collision>
-            <origin xyz="0 0 0" rpy="0 0 0" />
-            <geometry>
-                <mesh filename="package://dofbot_description/meshes/sensor/visual/mono_link.STL" />
+            <origin xyz="5.8458E-05 0.0095015 -0.0014824" rpy="0 0 0"/>
+            <mass value="0.0097589"/>
+            <inertia ixx="3.3488E-06" ixy="1.3667E-08" ixz="6.4235E-09" iyy="1.8662E-06" iyz="-1.0265E-07"
+                     izz="2.5696E-06"/>
+        </inertial>
+        <visual>
+            <origin xyz="0 0 0" rpy="0 0 0"/>
+            <geometry>
+                <mesh filename="package://dofbot_description/meshes/sensor/visual/mono_link.STL"/>
+            </geometry>
+            <material name="">
+                <color rgba="0.7 0.7 0.7 1"/>
+            </material>
+        </visual>
+        <collision>
+            <origin xyz="0 0 0" rpy="0 0 0"/>
+            <geometry>
+                <mesh filename="package://dofbot_description/meshes/sensor/visual/mono_link.STL"/>
             </geometry>
         </collision>
     </link>
     <joint name="mono_joint" type="fixed">
-        <origin xyz="-0.0481 -0.05145 -0.0022" rpy="1.5708 0 0" />
-        <parent link="arm_link_04" />
-        <child link="mono_link" />
-    </joint>
- <!--Trasmisión-->
-    <transmission name="trans_arm_joint_01">
-        <type>transmission_interface/SimpleTransmission</type>
-        <joint name="arm_joint_01">
-            <hardwareInterface>hardware_interface/PositionJointInterface</hardwareInterface>
-        </joint>
-        <actuator name="arm_joint_01_motor">
-            <hardwareInterface>hardware_interface/PositionJointInterface</hardwareInterface>
-            <mechanicalReduction>1</mechanicalReduction>
-        </actuator>
-    </transmission>
-    <transmission name="trans_arm_joint_02">
-        <type>transmission_interface/SimpleTransmission</type>
-        <joint name="arm_joint_02">
-            <hardwareInterface>hardware_interface/PositionJointInterface</hardwareInterface>
-        </joint>
-        <actuator name="arm_joint_02_motor">
-            <hardwareInterface>hardware_interface/PositionJointInterface</hardwareInterface>
-            <mechanicalReduction>1</mechanicalReduction>
-        </actuator>
-    </transmission>
-    <transmission name="trans_arm_joint_03">
-        <type>transmission_interface/SimpleTransmission</type>
-        <joint name="arm_joint_03">
-            <hardwareInterface>hardware_interface/PositionJointInterface</hardwareInterface>
-        </joint>
-        <actuator name="arm_joint_03_motor">
-            <hardwareInterface>hardware_interface/PositionJointInterface</hardwareInterface>
-            <mechanicalReduction>1</mechanicalReduction>
-        </actuator>
-    </transmission>
-    <transmission name="trans_arm_joint_04">
-        <type>transmission_interface/SimpleTransmission</type>
-        <joint name="arm_joint_04">
-            <hardwareInterface>hardware_interface/PositionJointInterface</hardwareInterface>
-        </joint>
-        <actuator name="arm_joint_04_motor">
-            <hardwareInterface>hardware_interface/PositionJointInterface</hardwareInterface>
-            <mechanicalReduction>1</mechanicalReduction>
-        </actuator>
-    </transmission>
-    <transmission name="trans_arm_joint_05">
-        <type>transmission_interface/SimpleTransmission</type>
-        <joint name="arm_joint_05">
-            <hardwareInterface>hardware_interface/PositionJointInterface</hardwareInterface>
-        </joint>
-        <actuator name="arm_joint_05_motor">
-            <hardwareInterface>hardware_interface/PositionJointInterface</hardwareInterface>
-            <mechanicalReduction>1</mechanicalReduction>
-        </actuator>
-    </transmission>
-    <transmission name="trans_grip_joint">
-        <type>transmission_interface/SimpleTransmission</type>
-        <joint name="grip_joint">
-            <hardwareInterface>hardware_interface/PositionJointInterface</hardwareInterface>
-        </joint>
-        <actuator name="grip_joint_motor">
-            <hardwareInterface>hardware_interface/PositionJointInterface</hardwareInterface>
-            <mechanicalReduction>1</mechanicalReduction>
-        </actuator>
-    </transmission>
-    <transmission name="trans_rfinger_joint_01">
-        <type>transmission_interface/SimpleTransmission</type>
-        <joint name="rfinger_joint_01">
-            <hardwareInterface>hardware_interface/PositionJointInterface</hardwareInterface>
-        </joint>
-        <actuator name="rfinger_joint_01_motor">
-            <hardwareInterface>hardware_interface/PositionJointInterface</hardwareInterface>
-            <mechanicalReduction>1</mechanicalReduction>
-        </actuator>
-    </transmission>
-    <transmission name="trans_rfinger_joint_02">
-        <type>transmission_interface/SimpleTransmission</type>
-        <joint name="rfinger_joint_02">
-            <hardwareInterface>hardware_interface/PositionJointInterface</hardwareInterface>
-        </joint>
-        <actuator name="rfinger_joint_02_motor">
-            <hardwareInterface>hardware_interface/PositionJointInterface</hardwareInterface>
-            <mechanicalReduction>1</mechanicalReduction>
-        </actuator>
-    </transmission>
-    <transmission name="trans_lfinger_grip_joint_01">
-        <type>transmission_interface/SimpleTransmission</type>
-        <joint name="lfinger_grip_joint_01">
-            <hardwareInterface>hardware_interface/PositionJointInterface</hardwareInterface>
-        </joint>
-        <actuator name="lfinger_grip_joint_01_motor">
-            <hardwareInterface>hardware_interface/PositionJointInterface</hardwareInterface>
-            <mechanicalReduction>1</mechanicalReduction>
-        </actuator>
-    </transmission>
-    <transmission name="trans_lfinger_grip_joint_02">
-        <type>transmission_interface/SimpleTransmission</type>
-        <joint name="lfinger_grip_joint_02">
-            <hardwareInterface>hardware_interface/EffortJointInterface</hardwareInterface>
-        </joint>
-        <actuator name="lfinger_grip_joint_02_motor">
-            <hardwareInterface>hardware_interface/EffortJointInterface</hardwareInterface>
-            <mechanicalReduction>1</mechanicalReduction>
-        </actuator>
-    </transmission>
-    <transmission name="trans_lfinger_grip_joint_03">
-        <type>transmission_interface/SimpleTransmission</type>
-        <joint name="lfinger_grip_joint_03">
-            <hardwareInterface>hardware_interface/PositionJointInterface</hardwareInterface>
-        </joint>
-        <actuator name="lfinger_grip_joint_03_motor">
-            <hardwareInterface>hardware_interface/PositionJointInterface</hardwareInterface>
-            <mechanicalReduction>1</mechanicalReduction>
-        </actuator>
-    </transmission>
- <!--Pluging control-->
-    <gazebo>
-        <plugin name="control" filename="libgazebo_ros_control.so"/>
-    </gazebo>
+        <origin xyz="-0.0481 -0.05145 -0.0022" rpy="1.5708 0 0"/>
+        <parent link="arm_link_04"/>
+        <child link="mono_link"/>
+    </joint>
+<!--
+    <joint name="mono_joint" type="revolute">
+        <origin xyz="-0.0481 -0.05145 -0.0022" rpy="1.5708 0 0"/>
+        <parent link="arm_link_04"/>
+        <child link="mono_link"/>
+        <axis xyz="0 0 1" />
+        <limit lower="0" upper="0" effort="0" velocity="0" />
+    </joint>-->
 </robot>

Commit message: Modify the fofbot launch file, add the driver for the gripper and updated config for the dofbot

File: dofbot_description/urdf/dofbot_arm_urdf.xacro (robot description, xacro)
@@ -390,15 +390,7 @@
     </link>
     <joint name="mono_joint" type="fixed">
-        <origin xyz="-0.0481 -0.05145 -0.0022" rpy="1.5708 0 0"/>
+        <origin xyz="-0.0482 -0.05145 -0.0022" rpy="1.5708 0 0"/>
         <parent link="arm_link_04"/>
         <child link="mono_link"/>
     </joint>
-<!--
-    <joint name="mono_joint" type="revolute">
-        <origin xyz="-0.0481 -0.05145 -0.0022" rpy="1.5708 0 0"/>
-        <parent link="arm_link_04"/>
-        <child link="mono_link"/>
-        <axis xyz="0 0 1" />
-        <limit lower="0" upper="0" effort="0" velocity="0" />
-    </joint>-->
 </robot>

Commit message: reordering urdf files and adding xacro_properties.xacro file to dofbot_description

File: dofbot_description/urdf/dofbot_arm_urdf.xacro (robot description, xacro)
@@ -365,32 +365,3 @@
         <mimic joint="grip_joint" multiplier="-1" />
     </joint>
-    <!-- Mono - camera sensor -->
-    <link name="mono_link">
-        <inertial>
-            <origin xyz="5.8458E-05 0.0095015 -0.0014824" rpy="0 0 0"/>
-            <mass value="0.0097589"/>
-            <inertia ixx="3.3488E-06" ixy="1.3667E-08" ixz="6.4235E-09" iyy="1.8662E-06" iyz="-1.0265E-07"
-                     izz="2.5696E-06"/>
-        </inertial>
-        <visual>
-            <origin xyz="0 0 0" rpy="0 0 0"/>
-            <geometry>
-                <mesh filename="package://dofbot_description/meshes/sensor/visual/mono_link.STL"/>
-            </geometry>
-            <material name="">
-                <color rgba="0.7 0.7 0.7 1"/>
-            </material>
-        </visual>
-        <collision>
-            <origin xyz="0 0 0" rpy="0 0 0"/>
-            <geometry>
-                <mesh filename="package://dofbot_description/meshes/sensor/visual/mono_link.STL"/>
-            </geometry>
-        </collision>
-    </link>
-    <joint name="mono_joint" type="fixed">
-        <origin xyz="-0.0482 -0.05145 -0.0022" rpy="1.5708 0 0"/>
-        <parent link="arm_link_04"/>
-        <child link="mono_link"/>
-    </joint>
 </robot>

File: dofbot_description/urdf/dofbot_trajectory_controller.xacro (robot description, xacro)
@@ -5,4 +5,5 @@
     <xacro:include filename="$(find ${package_name})/urdf/dofbot_gz_properties.xacro"/>
     <xacro:include filename="$(find ${package_name})/urdf/trajectory_controller.xacro"/>
+    <xacro:include filename="$(find ${package_name})/urdf/xacro_properties.xacro"/>
     <xacro:include filename="$(find ${package_name})/urdf/monocular_camera_sensor.xacro"/>
 </robot>

File: dofbot_description/urdf/monocular_camera_sensor.xacro (robot description, xacro)
@@ -1,11 +1,40 @@
 <?xml version="1.0" encoding="utf-8"?>
 <robot name="dofbot_camera" xmlns:xacro="http://ros.org/wiki/xacro" >
-    <link name="monocular_camera_link">
-    </link>
-    <joint name="base_camera_joint" type="fixed">
-        <parent link="mono_link" />
-        <child link="monocular_camera_link" />
-        <origin xyz="0 0 0" rpy="3.14 -1.57 0"/>
-    </joint>
+  <!-- Mono - camera sensor -->
+  <link name="mono_link">
+      <inertial>
+          <origin xyz="5.8458E-05 0.0095015 -0.0014824" rpy="0 0 0"/>
+          <mass value="0.0097589"/>
+          <inertia ixx="3.3488E-06" ixy="1.3667E-08" ixz="6.4235E-09" iyy="1.8662E-06" iyz="-1.0265E-07"
+                    izz="2.5696E-06"/>
+      </inertial>
+      <visual>
+          <origin xyz="0 0 0" rpy="0 0 0"/>
+          <geometry>
+              <mesh filename="package://dofbot_description/meshes/sensor/visual/mono_link.STL"/>
+          </geometry>
+          <material name="">
+              <color rgba="0.7 0.7 0.7 1"/>
+          </material>
+      </visual>
+      <collision>
+          <origin xyz="0 0 0" rpy="0 0 0"/>
+          <geometry>
+              <mesh filename="package://dofbot_description/meshes/sensor/visual/mono_link.STL"/>
+          </geometry>
+      </collision>
+  </link>
+  <joint name="mono_joint" type="fixed">
+      <origin xyz="${mono_joint_xyz}" rpy="${mono_joint_rpy}"/>
+      <parent link="arm_link_04"/>
+      <child link="mono_link"/>
+  </joint>
+  <link name="monocular_camera_link">
+  </link>
+  <joint name="base_camera_joint" type="fixed">
+      <parent link="mono_link" />
+      <child link="monocular_camera_link" />
+      <origin xyz="0 0 0" rpy="3.14 -1.57 0"/>
+  </joint>
   <!-- MONOCULAR CAMERA -->
   <gazebo reference="monocular_camera_link">
