Commit message: added new stl, update xacro_properties and URDF refactor

File: dofbot_description/urdf/dofbot_arm_urdf.xacro (robot description, xacro)
@@ -19,24 +19,5 @@
  <!--Dofbot description-->
     <!--Dofbot Arm Base Link-->
-    <link name="arm_base_link">
-        <visual>
-            <origin xyz="0.0 0.0 0.0" rpy="0.0 0.0 0.0" />
-            <geometry>
-                <mesh filename="package://dofbot_description/meshes/dofbot/visual/base_link.STL" />
-            </geometry>
-            <material name="eerie_black" />
-        </visual>
-        <collision>
-            <origin xyz="0.0 0.0 0.0" rpy="0.0 0.0 0.0" />
-            <geometry>
-                <mesh filename="package://dofbot_description/meshes/dofbot/visual/base_link.STL" />
-            </geometry>
-        </collision>
-        <inertial>
-            <origin xyz="-0.0304416859098744 4.23384368655101E-05 0.0448234503408059" rpy="0 0 0" />
-            <mass value="1.0754239466482" />
-            <inertia ixx="0.0208831789264125" ixy="2.4618093127858E-06" ixz="0.00616019290028669" iyy="0.0265621377486244" iyz="-1.10079499865282E-06" izz="0.0129535610833954" />
-        </inertial>
-    </link>
+    <xacro:include filename="$(find ${package_name})/urdf/arm_base_link_xacro.xacro"/>
     <!-- Dofbot Arm Link 01 -->
     <link name="arm_link_01">

File: omni_description/urdf/omni_urdf.xacro (robot description, xacro)
@@ -15,7 +15,7 @@
         </inertial>
         <visual>
-            <origin xyz="0 0 0" rpy="0 0 0"/>
+            <origin xyz="${base_link_xyz}" rpy="0 0 0"/>
             <geometry>
-                <mesh filename="package://omni_description/meshes/X3/base_link.STL"/>
+                <mesh filename="${base_mesh}"/>
             </geometry>
             <material name="">
@@ -24,7 +24,7 @@
         </visual>
         <collision>
-            <origin xyz="0 0 0" rpy="0 0 0"/>
+            <origin xyz="${base_link_xyz}" rpy="0 0 0"/>
             <geometry>
-                <mesh filename="package://omni_description/meshes/X3/base_link.STL"/>
+                <mesh filename="${base_mesh}"/>
             </geometry>
         </collision>
@@ -45,5 +45,5 @@
             <origin xyz="0 0 0" rpy="0 0 0"/>
             <geometry>
-                <mesh filename="package://omni_description/meshes/X3/front_right_wheel.STL"/>
+                <mesh filename="${f_r_wheel}"/>
             </geometry>
             <material name="">
@@ -54,10 +54,10 @@
             <origin xyz="0 0 0" rpy="0 0 0"/>
             <geometry>
-                <mesh filename="package://omni_description/meshes/X3/front_right_wheel.STL"/>
+                <mesh filename="${f_r_wheel}"/>
             </geometry>
         </collision>
     </link>
     <joint name="front_right_joint" type="continuous">
-        <origin xyz="0.08 -0.0845 -0.0389" rpy="-1.5703 0 3.14159"/>
+        <origin xyz="${f_r_wheel_xyz}" rpy="-1.5703 0 3.14159"/>
         <parent link="base_link"/>
         <child link="front_right_wheel"/>
@@ -75,5 +75,5 @@
             <origin xyz="0 0 0" rpy="0 0 0"/>
             <geometry>
-                <mesh filename="package://omni_description/meshes/X3/front_left_wheel.STL"/>
+                <mesh filename="${f_l_wheel}"/>
             </geometry>
             <material name="">
@@ -84,10 +84,10 @@
             <origin xyz="0 0 0" rpy="0 0 0"/>
             <geometry>
-                <mesh filename="package://omni_description/meshes/X3/front_left_wheel.STL"/>
+                <mesh filename="${f_l_wheel}"/>
             </geometry>
         </collision>
     </link>
     <joint name="front_left_joint" type="continuous">
-        <origin xyz="0.08 0.084492 -0.0389" rpy="1.5703 0 0"/>
+        <origin xyz="${f_l_wheel_xyz}" rpy="1.5703 0 0"/>
         <parent link="base_link"/>
         <child link="front_left_wheel"/>
@@ -105,5 +105,5 @@
             <origin xyz="0 0 0" rpy="0 0 0"/>
             <geometry>
-                <mesh filename="package://omni_description/meshes/X3/back_right_wheel.STL"/>
+                <mesh filename="${b_r_wheel}"/>
             </geometry>
             <material name="">
@@ -114,10 +114,10 @@
             <origin xyz="0 0 0" rpy="0 0 0"/>
             <geometry>
-                <mesh filename="package://omni_description/meshes/X3/back_right_wheel.STL"/>
+                <mesh filename="${b_r_wheel}"/>
             </geometry>
         </collision>
     </link>
     <joint name="back_right_joint" type="continuous">
-        <origin xyz="-0.08 -0.0845 -0.03946" rpy="-1.57 0 3.14159"/>
+        <origin xyz="${b_r_wheel_xyz}" rpy="-1.57 0 3.14159"/>
         <parent link="base_link"/>
         <child link="back_right_wheel"/>
@@ -135,5 +135,5 @@
             <origin xyz="0 0 0" rpy="0 0 0"/>
             <geometry>
-                <mesh filename="package://omni_description/meshes/X3/back_left_wheel.STL"/>
+                <mesh filename="${b_l_wheel}"/>
             </geometry>
             <material name="">
@@ -144,10 +144,10 @@
             <origin xyz="0 0 0" rpy="0 0 0"/>
             <geometry>
-                <mesh filename="package://omni_description/meshes/X3/back_left_wheel.STL"/>
+                <mesh filename="${b_l_wheel}"/>
             </geometry>
         </collision>
     </link>
     <joint name="back_left_joint" type="continuous">
-        <origin xyz="-0.08 0.084492 -0.03954" rpy="1.5703 0 0"/>
+        <origin xyz="${b_l_wheel_xyz}" rpy="1.5703 0 0"/>
         <parent link="base_link"/>
         <child link="back_left_wheel"/>

File: omni_description/urdf/omni_velocity_controller.xacro (robot description, xacro)
@@ -2,8 +2,8 @@
 <robot name="Omni_bot" xmlns:xacro="http://ros.org/wiki/xacro">
     <xacro:property name="package_name" value="omni_description" />
+    <xacro:include filename="$(find ${package_name})/urdf/xacro_properties.xacro"/>
     <xacro:include filename="$(find ${package_name})/urdf/omni_urdf.xacro"/>
     <xacro:include filename="$(find ${package_name})/urdf/omni_gz_properties.xacro"/>
     <xacro:include filename="$(find ${package_name})/urdf/velocity_controller.xacro"/>
-    <xacro:include filename="$(find ${package_name})/urdf/xacro_properties.xacro"/>
     <xacro:include filename="$(find ${package_name})/urdf/lidar_sensor.xacro"/>
     <xacro:include filename="$(find ${package_name})/urdf/camera_sensor.xacro"/>

File: omni_description/urdf/xacro_properties.xacro (robot description, xacro)
@@ -7,3 +7,13 @@
     <xacro:property name="imu_joint_xyz" value="-0.06 0.01 0.01"/>
     <xacro:property name="imu_joint_rpy" value="0 3.1415 1.5707"/>
+    <xacro:property name="base_link_xyz" value="0 0 0"/>
+    <xacro:property name="base_mesh" value="package://omni_description/meshes/X3/base_link.STL"/>
+    <xacro:property name="f_l_wheel_xyz" value="0.08 0.084492 -0.0389"/>
+    <xacro:property name="f_r_wheel_xyz" value="0.08 -0.0845 -0.0389"/>
+    <xacro:property name="b_l_wheel_xyz" value="-0.08 0.084492 -0.03954"/>
+    <xacro:property name="b_r_wheel_xyz" value="-0.08 -0.0845 -0.03946"/>
+    <xacro:property name="f_l_wheel" value="package://omni_description/meshes/X3/front_left_wheel.STL"/>
+    <xacro:property name="f_r_wheel" value="package://omni_description/meshes/X3/front_right_wheel.STL"/>
+    <xacro:property name="b_l_wheel" value="package://omni_description/meshes/X3/back_left_wheel.STL"/>
+    <xacro:property name="b_r_wheel" value="package://omni_description/meshes/X3/back_right_wheel.STL"/>
 </robot>

File: omni_dofbot_description/urdf/omni_dofbot_urdf.xacro (robot description, xacro)
@@ -1,17 +1,63 @@
 <?xml version="1.0" encoding="UTF-8" ?>
 <robot name="omni_dofbot" xmlns:xacro="http://ros.org/wiki/xacro">
+  <xacro:include filename="$(find omni_dofbot_description)/urdf/xacro_properties.xacro" />
   <xacro:include filename="$(find omni_description)/urdf/omni_urdf.xacro" />
   <!--
   <xacro:include filename="$(find omni_dofbot_description)/urdf/dofbot_without_base_urdf.xacro" />-->
   <xacro:include filename="$(find dofbot_description)/urdf/dofbot_arm_urdf.xacro" />
-  <xacro:include filename="$(find omni_dofbot_description)/urdf/xacro_properties.xacro" />
   <xacro:include filename="$(find omni_description)/urdf/camera_sensor.xacro" />
   <xacro:include filename="$(find omni_description)/urdf/lidar_sensor.xacro" />
   <xacro:include filename="$(find dofbot_description)/urdf/monocular_camera_sensor.xacro"/>
   <xacro:include filename="$(find omni_description)/urdf/imu_sensor.xacro"/>
-  <joint name="omni_to_dofbot_joint" type="fixed">
+  <joint name="omni_to_dofbot_joint" type="revolute">
     <parent link="base_link" />
     <child link="arm_base_link" />
-    <origin xyz="0.045 0 0.055" rpy="0 0 -1.57" />
+    <origin xyz="0.1025 0 0.031" rpy="0 0 -1.57" />
+    <axis xyz="0 0 1" />
+    <limit lower="0" upper="0" effort="1" velocity="1" />
+  </joint>
+  <link name="mastil_link">
+    <visual>
+      <origin xyz="0 0 ${0.355/2}" rpy="0 0 0"/>
+      <geometry>
+        <box size="0.02 0.04 0.355"/>
+      </geometry>
+      <material name="black">
+        <color rgba="0 0 0 1.0"/>
+      </material>
+    </visual>
+    <collision>
+      <origin rpy="0 0 0" xyz="0 0 ${0.355/2}"/>
+      <geometry>
+        <box size="0.02 0.04 0.355"/>
+      </geometry>
+    </collision>
+  </link>
+  <joint name="base_to_mastil_joint" type="fixed">
+    <origin xyz="-0.035 0 0.0615" rpy="0 0 0"/>
+    <parent link="base_link"/>
+    <child link="mastil_link"/>
+  </joint>
+  <link name="display_link">
+    <visual>
+      <origin rpy="0 0 0" xyz="0 0 0"/>
+      <geometry>
+        <mesh filename="package://omni_dofbot_description/meshes/display_omni_dofbot.stl"/>
+      </geometry>
+      <material name="">
+        <color rgba="0 0.7 0 1"/>
+      </material>
+    </visual>
+    <collision>
+      <origin rpy="0 0 0" xyz="0 0 0"/>
+      <geometry>
+        <mesh filename="package://omni_dofbot_description/meshes/display_omni_dofbot.stl"/>
+      </geometry>
+    </collision>
+  </link>
+  <joint name="display_joint" type="fixed">
+    <parent link="mastil_link"/>
+    <child link="display_link"/>
+    <origin rpy="0 0 0" xyz="-0.07 0.0 0.265"/>
   </joint>
 </robot>

File: omni_dofbot_description/urdf/xacro_properties.xacro (robot description, xacro)
@@ -1,7 +1,7 @@
 <?xml version="1.0" encoding="utf-8"?>
 <robot xmlns:xacro="http://ros.org/wiki/xacro" >
-    <xacro:property name="laser_joint_xyz" value="0.057105 1.7948E-05 0.03755"/>
+    <xacro:property name="laser_joint_xyz" value="0.11 1.7948E-05 0.03755"/>
     <xacro:property name="laser_joint_rpy" value="0.0 0.0 0.0"/>
-    <xacro:property name="camera_joint_xyz" value="-0.05 0.01 0.51"/>
+    <xacro:property name="camera_joint_xyz" value="-0.035 0.00 0.45"/>
     <xacro:property name="camera_joint_rpy" value="0.0 0.0 0.0"/>
     <xacro:property name="imu_joint_xyz" value="-0.06 0.01 0.01"/>
@@ -9,3 +9,13 @@
     <xacro:property name="mono_joint_xyz" value="-0.0482 -0.05145 -0.0022"/>
     <xacro:property name="mono_joint_rpy" value="1.5708 0 0"/>
+    <xacro:property name="base_link_xyz" value="0.05 0 0.02"/>
+    <xacro:property name="base_mesh" value="package://omni_dofbot_description/meshes/base_link_omni_dofbot.stl"/>
+    <xacro:property name="f_l_wheel_xyz" value="0.11 0.099492 -0.0389"/>
+    <xacro:property name="f_r_wheel_xyz" value="0.11 -0.1045 -0.0389"/>
+    <xacro:property name="b_l_wheel_xyz" value="-0.11 0.100492 -0.03954"/>
+    <xacro:property name="b_r_wheel_xyz" value="-0.11 -0.1005 -0.03946"/>
+    <xacro:property name="f_l_wheel" value="package://omni_dofbot_description/meshes/80mm_mecanum_wheel_hex.stl"/>
+    <xacro:property name="f_r_wheel" value="package://omni_dofbot_description/meshes/80mm_mecanum_wheel_hex.stl"/>
+    <xacro:property name="b_l_wheel" value="package://omni_dofbot_description/meshes/80mm_mecanum_wheel_hex.stl"/>
+    <xacro:property name="b_r_wheel" value="package://omni_dofbot_description/meshes/80mm_mecanum_wheel_hex.stl"/>
 </robot>
