Commit message: Updated omni_dofbot_urdf.xacro file

File: omni_dofbot_description/urdf/omni_dofbot_urdf.xacro (robot description, xacro)
@@ -2,9 +2,143 @@
 <robot name="omni_dofbot" xmlns:xacro="http://ros.org/wiki/xacro">
   <xacro:include filename="$(find omni_description)/urdf/omni_urdf.xacro" />
+  <!--
+  <xacro:include filename="$(find omni_dofbot_description)/urdf/dofbot_without_base_urdf.xacro" />-->
   <xacro:include filename="$(find dofbot_description)/urdf/dofbot_arm_urdf.xacro" />
+  <xacro:include filename="$(find omni_description)/urdf/camera_sensor.xacro" />
+  <xacro:include filename="$(find omni_description)/urdf/lidar_sensor.xacro" />
+  <xacro:include filename="$(find dofbot_description)/urdf/monocular_camera_sensor.xacro"/>
+  <xacro:include filename="$(find omni_description)/urdf/imu_sensor.xacro"/>
   <joint name="omni_to_dofbot_joint" type="fixed">
     <parent link="base_link" />
     <child link="arm_base_link" />
-    <origin xyz="0.1 0 0.15" rpy="0 0 -1.57" />
+    <origin xyz="0.045 0 0.055" rpy="0 0 -1.57" />
   </joint>
+  <ros2_control name="GazeboSystem_dofbot" type="system">
+      <hardware>
+          <plugin>gazebo_ros2_control/GazeboSystem</plugin>
+      </hardware>
+      <joint name="arm_joint_01">
+          <command_interface name="position"/>
+          <state_interface name="position"/>
+          <state_interface name="velocity"/>
+          <state_interface name="effort"/>
+      </joint>
+      <joint name="arm_joint_02">
+          <command_interface name="position"/>
+          <state_interface name="position"/>
+          <state_interface name="velocity"/>
+          <state_interface name="effort"/>
+      </joint>
+      <joint name="arm_joint_03">
+          <command_interface name="position"/>
+          <state_interface name="position"/>
+          <state_interface name="velocity"/>
+          <state_interface name="effort"/>
+      </joint>
+      <joint name="arm_joint_04">
+          <command_interface name="position"/>
+          <state_interface name="position"/>
+          <state_interface name="velocity"/>
+          <state_interface name="effort"/>
+      </joint>
+      <joint name="arm_joint_05">
+          <command_interface name="position"/>
+          <state_interface name="position"/>
+          <state_interface name="velocity"/>
+          <state_interface name="effort"/>
+      </joint>
+      <joint name="grip_joint">
+          <command_interface name="position"/>
+          <state_interface name="position"/>
+          <state_interface name="velocity"/>
+          <state_interface name="effort"/>
+      </joint>
+      <joint name="rfinger_joint_01">
+          <command_interface name="position"/>
+          <state_interface name="position"/>
+          <state_interface name="velocity"/>
+          <state_interface name="effort"/>
+      </joint>
+      <joint name="rfinger_joint_02">
+          <command_interface name="position"/>
+          <state_interface name="position"/>
+          <state_interface name="velocity"/>
+          <state_interface name="effort"/>
+      </joint>
+      <joint name="lfinger_grip_joint_01">
+          <command_interface name="position"/>
+          <state_interface name="position"/>
+          <state_interface name="velocity"/>
+          <state_interface name="effort"/>
+      </joint>
+      <joint name="lfinger_grip_joint_02">
+          <command_interface name="position"/>
+          <state_interface name="position"/>
+          <state_interface name="velocity"/>
+          <state_interface name="effort"/>
+      </joint>
+      <joint name="lfinger_grip_joint_03">
+          <command_interface name="position"/>
+          <state_interface name="position"/>
+          <state_interface name="velocity"/>
+          <state_interface name="effort"/>
+      </joint>
+      <joint name="front_left_joint"> <!-- M1 -->
+        <command_interface name="velocity"/>
+        <state_interface name="position"/>
+        <state_interface name="velocity"/>
+        <state_interface name="effort"/>
+      </joint>
+      <joint name="front_right_joint"> <!-- M2 -->
+        <command_interface name="velocity"/>
+        <state_interface name="position"/>
+        <state_interface name="velocity"/>
+        <state_interface name="effort"/>
+      </joint>
+      <joint name="back_right_joint"> <!-- M3 -->
+        <command_interface name="velocity"/>
+        <state_interface name="position"/>
+        <state_interface name="velocity"/>
+        <state_interface name="effort"/>
+      </joint>
+      <joint name="back_left_joint"> <!-- M4 -->
+        <command_interface name="velocity"/>
+        <state_interface name="position"/>
+        <state_interface name="velocity"/>
+        <state_interface name="effort"/>
+      </joint>
+  </ros2_control>
+  <!-- Omnidirectional plugin -->
+  <gazebo>
+    <plugin name="omni_controller_gz" filename="libgazebo_ros_planar_move.so"> <!-- 3 DOF plugin, (Vx,Vy,Wz) -->
+      <command_topic>cmd_vel</command_topic>
+      <odometry_topic>odom</odometry_topic>
+      <odometry_frame>odom</odometry_frame>
+      <robot_base_frame>base_footprint</robot_base_frame>
+      <publish_odom>true</publish_odom>
+      <publish_odom_tf>true</publish_odom_tf>
+      <update_rate>30</update_rate>
+    </plugin>
+  </gazebo>
+  <!-- Plugin para visualizar correctamente las posiciones de las juntas en RViz -->
+  <gazebo>
+    <plugin name="joint_states_gz" filename="libgazebo_ros_joint_state_publisher.so">
+      <ros>
+        <remapping>~/out:=joint_states</remapping>
+      </ros>
+      <update_rate>30</update_rate>
+      <joint_name>front_left_joint</joint_name>
+      <joint_name>front_right_joint</joint_name>
+      <joint_name>back_right_joint</joint_name>
+      <joint_name>back_left_joint</joint_name>
+    </plugin>
+  </gazebo>
+  <!-- Plugin de control ROS 2 -->
+  <gazebo>
+    <plugin name="gazebo_ros2_control" filename="libgazebo_ros2_control.so">
+      <robot_param>robot_description</robot_param>
+      <robot_param_node>robot_state_publisher</robot_param_node>
+      <parameters>$(find omni_dofbot_description)/config/omni_dofbot_controller.yaml</parameters>
+    </plugin>
+  </gazebo>
 </robot>

Commit message: I split the file omni_dofbot_urfd.xacro

File: omni_dofbot_description/urdf/omni_dofbot_urdf.xacro (robot description, xacro)
@@ -14,131 +14,3 @@
     <origin xyz="0.045 0 0.055" rpy="0 0 -1.57" />
   </joint>
-  <ros2_control name="GazeboSystem_dofbot" type="system">
-      <hardware>
-          <plugin>gazebo_ros2_control/GazeboSystem</plugin>
-      </hardware>
-      <joint name="arm_joint_01">
-          <command_interface name="position"/>
-          <state_interface name="position"/>
-          <state_interface name="velocity"/>
-          <state_interface name="effort"/>
-      </joint>
-      <joint name="arm_joint_02">
-          <command_interface name="position"/>
-          <state_interface name="position"/>
-          <state_interface name="velocity"/>
-          <state_interface name="effort"/>
-      </joint>
-      <joint name="arm_joint_03">
-          <command_interface name="position"/>
-          <state_interface name="position"/>
-          <state_interface name="velocity"/>
-          <state_interface name="effort"/>
-      </joint>
-      <joint name="arm_joint_04">
-          <command_interface name="position"/>
-          <state_interface name="position"/>
-          <state_interface name="velocity"/>
-          <state_interface name="effort"/>
-      </joint>
-      <joint name="arm_joint_05">
-          <command_interface name="position"/>
-          <state_interface name="position"/>
-          <state_interface name="velocity"/>
-          <state_interface name="effort"/>
-      </joint>
-      <joint name="grip_joint">
-          <command_interface name="position"/>
-          <state_interface name="position"/>
-          <state_interface name="velocity"/>
-          <state_interface name="effort"/>
-      </joint>
-      <joint name="rfinger_joint_01">
-          <command_interface name="position"/>
-          <state_interface name="position"/>
-          <state_interface name="velocity"/>
-          <state_interface name="effort"/>
-      </joint>
-      <joint name="rfinger_joint_02">
-          <command_interface name="position"/>
-          <state_interface name="position"/>
-          <state_interface name="velocity"/>
-          <state_interface name="effort"/>
-      </joint>
-      <joint name="lfinger_grip_joint_01">
-          <command_interface name="position"/>
-          <state_interface name="position"/>
-          <state_interface name="velocity"/>
-          <state_interface name="effort"/>
-      </joint>
-      <joint name="lfinger_grip_joint_02">
-          <command_interface name="position"/>
-          <state_interface name="position"/>
-          <state_interface name="velocity"/>
-          <state_interface name="effort"/>
-      </joint>
-      <joint name="lfinger_grip_joint_03">
-          <command_interface name="position"/>
-          <state_interface name="position"/>
-          <state_interface name="velocity"/>
-          <state_interface name="effort"/>
-      </joint>
-      <joint name="front_left_joint"> <!-- M1 -->
-        <command_interface name="velocity"/>
-        <state_interface name="position"/>
-        <state_interface name="velocity"/>
-        <state_interface name="effort"/>
-      </joint>
-      <joint name="front_right_joint"> <!-- M2 -->
-        <command_interface name="velocity"/>
-        <state_interface name="position"/>
-        <state_interface name="velocity"/>
-        <state_interface name="effort"/>
-      </joint>
-      <joint name="back_right_joint"> <!-- M3 -->
-        <command_interface name="velocity"/>
-        <state_interface name="position"/>
-        <state_interface name="velocity"/>
-        <state_interface name="effort"/>
-      </joint>
-      <joint name="back_left_joint"> <!-- M4 -->
-        <command_interface name="velocity"/>
-        <state_interface name="position"/>
-        <state_interface name="velocity"/>
-        <state_interface name="effort"/>
-      </joint>
-  </ros2_control>
-  <!-- Omnidirectional plugin -->
-  <gazebo>
-    <plugin name="omni_controller_gz" filename="libgazebo_ros_planar_move.so"> <!-- 3 DOF plugin, (Vx,Vy,Wz) -->
-      <command_topic>cmd_vel</command_topic>
-      <odometry_topic>odom</odometry_topic>
-      <odometry_frame>odom</odometry_frame>
-      <robot_base_frame>base_footprint</robot_base_frame>
-      <publish_odom>true</publish_odom>
-      <publish_odom_tf>true</publish_odom_tf>
-      <update_rate>30</update_rate>
-    </plugin>
-  </gazebo>
-  <!-- Plugin para visualizar correctamente las posiciones de las juntas en RViz -->
-  <gazebo>
-    <plugin name="joint_states_gz" filename="libgazebo_ros_joint_state_publisher.so">
-      <ros>
-        <remapping>~/out:=joint_states</remapping>
-      </ros>
-      <update_rate>30</update_rate>
-      <joint_name>front_left_joint</joint_name>
-      <joint_name>front_right_joint</joint_name>
-      <joint_name>back_right_joint</joint_name>
-      <joint_name>back_left_joint</joint_name>
-    </plugin>
-  </gazebo>
-  <!-- Plugin de control ROS 2 -->
-  <gazebo>
-    <plugin name="gazebo_ros2_control" filename="libgazebo_ros2_control.so">
-      <robot_param>robot_description</robot_param>
-      <robot_param_node>robot_state_publisher</robot_param_node>
-      <parameters>$(find omni_dofbot_description)/config/omni_dofbot_controller.yaml</parameters>
-    </plugin>
-  </gazebo>
 </robot>

Commit message: The type of joint omni_to_dofbot_joint was changed to fixed and gazebo materials were added.

File: omni_dofbot_description/urdf/omni_dofbot_urdf.xacro (robot description, xacro)
@@ -1,4 +1,4 @@
 <?xml version="1.0" encoding="UTF-8" ?>
-<robot name="omni_dofbot" xmlns:xacro="http://ros.org/wiki/xacro">
+<robot name="omni_dofbot_urdf" xmlns:xacro="http://ros.org/wiki/xacro">
   <xacro:include filename="$(find omni_dofbot_description)/urdf/xacro_properties.xacro" />
   <xacro:include filename="$(find omni_description)/urdf/omni_urdf.xacro" />
@@ -10,10 +10,8 @@
   <xacro:include filename="$(find dofbot_description)/urdf/monocular_camera_sensor.xacro"/>
   <xacro:include filename="$(find omni_description)/urdf/imu_sensor.xacro"/>
-  <joint name="omni_to_dofbot_joint" type="revolute">
+  <joint name="omni_to_dofbot_joint" type="fixed">
+    <origin xyz="0.1025 0 0.031" rpy="0 0 -1.57" />
     <parent link="base_link" />
     <child link="arm_base_link" />
-    <origin xyz="0.1025 0 0.031" rpy="0 0 -1.57" />
-    <axis xyz="0 0 1" />
-    <limit lower="0" upper="0" effort="1" velocity="1" />
   </joint>
   <link name="mastil_link">
@@ -23,6 +21,6 @@
         <box size="0.02 0.04 0.355"/>
       </geometry>
-      <material name="black">
-        <color rgba="0 0 0 1.0"/>
+      <material name="grey">
+        <color rgba="0.5 0.5 0.5 1.0"/>
       </material>
     </visual>
@@ -61,3 +59,9 @@
     <origin rpy="0 0 0" xyz="-0.07 0.0 0.265"/>
   </joint>
+  <gazebo reference="mastil_link">
+    <material>Gazebo/Grey</material>
+  </gazebo>
+  <gazebo reference="display_link">
+    <material>Gazebo/BlueTransparent</material>
+  </gazebo>
 </robot>
