Commit message: Added inertial propertie in arm_base_link_xacro.xacro file

File: omni_dofbot_description/urdf/arm_base_link_xacro.xacro (robot description, xacro)
@@ -2,4 +2,7 @@
 <robot xmlns:xacro="http://ros.org/wiki/xacro">
     <link name="arm_base_link">
+        <inertial>
+            <mass value="0.0001" />
+        </inertial>
     </link>
 </robot>

Commit message: add origin and intertia to arm_base_link

File: omni_dofbot_description/urdf/arm_base_link_xacro.xacro (robot description, xacro)
@@ -4,4 +4,6 @@
         <inertial>
             <mass value="0.0001" />
+            <origin xyz="0 0 0" rpy="0 0 0" />
+            <inertia ixx="0" ixy="0" ixz="0" iyy="0" iyz="0" izz="0" />
         </inertial>
     </link>
